File: Hardware/InkTime.brd (EAGLE design)
At the start: 46 x 35 mm, 105 parts, among them IC1 BQ25180YBGR_BQ25180YBGR, IC2 DRV2605YZFR_DRV2605YZFR, IC3 BMA423_BMA423, IC9 RT6160AWSC_RT6160AWSC, J1 503480-2400_503480-2400, J2 TC2030-IDC_TC2030-IDC, J4 KH-TYPE-C-16P_KH-TYPE-C-16P, Q1 20V/4.2A/52mΩ/1.4W, Q3 ESP32_C6_LIBRARY_6_SI1308EDL-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, U1 NORDIC_NRF_4_NRF52840_QF, U3 ESP32_C6_LIBRARY_MAX17048G+T10, X1 32MHz, X2 32.768kHz

Commit message: added routes
Routing:
- net 3V3/2.4A: track 0.00 -> 130.3 mm, vias 0 -> 17
- net GND: track 0.00 -> 82.5 mm, vias 0 -> 2
- net PREVGH: track 0.00 -> 65.2 mm, vias 0 -> 2
- net EPD_3V3: track 0.00 -> 64.7 mm, vias 0 -> 4
- net SDA/2.4C: track 0.00 -> 61.0 mm, vias 0 -> 5
- net VBUS/2.6D: track 0.00 -> 50.7 mm, vias 0 -> 3
- net N$6: track 0.00 -> 49.7 mm, vias 0 -> 2
- net GDR: track 0.00 -> 49.6 mm, vias 0 -> 3
- net 3V3/1.7D: track 0.00 -> 49.0 mm, vias 0 -> 2
- net PREVGL: track 0.00 -> 48.9 mm, vias 0 -> 2
- net N$26: track 0.00 -> 48.3 mm, vias 0 -> 5
- net DN: track 0.00 -> 48.2 mm, vias 0 -> 3
- net VBUS/1.5D: track 0.00 -> 47.7 mm, vias 0 -> 9
- net DP: track 0.00 -> 46.1 mm, vias 0 -> 4
- net OUT-: track 0.00 -> 43.6 mm, vias 0 -> 2
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
Commit message: issue solved
Routing:
- net GND: track 82.5 -> 913.0 mm, vias 2 -> 31
